File: hardware/mote/rev_a/mote.sch (EAGLE design)
At the start: 139 parts, among them J1 TC2030-JLINK-L, J2 TC2030-JLINK-NL, Q1 CSD22206W, Q10 CSD22206W, Q11 CSD22206W, Q2 CSD22206W, Q6 CSD22206W, Q7 CSD22206W, Q8 CSD22206W, Q9 CSD22206W, U1 NRF52840, U10 MS5637-02BA03, U11 ADP5091, U12 NRF51822QF, U3 MAX17222, U4 AMN41121, U5 SI7021-A20-GM1, U6 ISL29125, U7 MAX44009, U8 LIS2DW12, U9 AB1815-T3, X1 7V-32.000MAHV-T, X2 ABS05-32.768KHZ-9-T, X3 ABS07-32.768KHZ-7-T, X5 16MHz, X6 ABS05-32.768KHZ-9-T

Commit message: route signals out of mcu
Parts:
- C26: DIGIKEY 490-3896-2-ND -> 490-4516-1-ND
Connections:
- removed net CLKOUT: U9.CLKOUT/!IRQ3
- new net !RTC_IRQ3: U1.P1.07, U9.CLKOUT/!IRQ3
- net !CLR_EN: now also U1.P0.11; no longer U1.P0.20
- net !I2C_EN: now also U1.P1.11
- net !RTC_IRQ1: now also U1.P0.14
- net !RTC_IRQ2: now also U1.P0.20
- net ACC_CS: now also U1.P0.13; no longer U1.P0.15
- net RTC_CS: now also U1.P0.15; no longer U1.P0.13
Other:
- note added: "AD12 is in the way of the actual Reset pin, AC13, so we just route over it."
Changed lines of the file:
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@@
 <part name="GND21" library="supply1" library_urn="urn:adsk.eagle:library:371" deviceset="GND" device=""/>
 <part name="C26" library="passives" deviceset="CAPACITOR" device="0603_CAP" value="10nF">
-<attribute name="DIGIKEY" value="490-3896-2-ND"/>
+<attribute name="DIGIKEY" value="490-4516-1-ND"/>
 </part>
 <part name="R21" library="passives" deviceset="RESISTOR" device="0402_RES" value="18MΩ"/>
@@
 <wire x1="99.06" y1="55.88" x2="99.06" y2="0" width="0.254" layer="94" style="shortdash"/>
 <text x="2.54" y="50.8" size="2.54" layer="97">RTC</text>
+<text x="66.04" y="81.28" size="1.27" layer="98">AD12 is in the way of the
+actual Reset pin, AC13,
+so we just route over it.</text>
 </plain>
 <instances>
@@
 </segment>
 </net>
-<net name="CLKOUT" class="0">
-<segment>
-<pinref part="U9" gate="G$1" pin="CLKOUT/!IRQ3"/>
-<wire x1="83.82" y1="27.94" x2="86.36" y2="27.94" width="0.1524" layer="91"/>
-<label x="86.36" y="27.94" size="1.27" layer="95" xref="yes"/>
-</segment>
-</net>
 <net name="SCL" class="0">
 <segment>
@@
 <label x="86.36" y="33.02" size="1.27" layer="95" xref="yes"/>
 </segment>
+<segment>
+<pinref part="U1" gate="G$1" pin="P0.14"/>
+<wire x1="99.06" y1="91.44" x2="93.98" y2="91.44" width="0.1524" layer="91"/>
+<label x="93.98" y="91.44" size="1.27" layer="95" rot="R180" xref="yes"/>
+</segment>
 </net>
 <net name="!RTC_IRQ2" class="0">
@@
 <wire x1="83.82" y1="30.48" x2="86.36" y2="30.48" width="0.1524" layer="91"/>
 <label x="86.36" y="30.48" size="1.27" layer="95" xref="yes"/>
+</segment>
+<segment>
+<pinref part="U1" gate="G$1" pin="P0.20"/>
+<wire x1="99.06" y1="78.74" x2="93.98" y2="78.74" width="0.1524" layer="91"/>
+<label x="93.98" y="78.74" size="1.27" layer="95" rot="R180" xref="yes"/>
 </segment>
 </net>
@@
 </segment>
 <segment>
-<pinref part="U1" gate="G$1" pin="P0.13"/>
-<wire x1="99.06" y1="93.98" x2="93.98" y2="93.98" width="0.1524" layer="91"/>
-<label x="93.98" y="93.98" size="1.27" layer="95" rot="R180" xref="yes"/>
+<pinref part="U1" gate="G$1" pin="P0.15"/>
+<wire x1="99.06" y1="88.9" x2="93.98" y2="88.9" width="0.1524" layer="91"/>
+<label x="93.98" y="88.9" size="1.27" layer="95" rot="R180" xref="yes"/>
 </segment>
 </net>
@@
 <wire x1="144.78" y1="91.44" x2="147.32" y2="91.44" width="0.1524" layer="91"/>
 <label x="147.32" y="91.44" size="1.27" layer="95" xref="yes"/>
-</segment>
-</net>
-<net name="!CLR_EN" class="0">
-<segment>
-<pinref part="U1" gate="G$1" pin="P0.20"/>
-<wire x1="99.06" y1="78.74" x2="93.98" y2="78.74" width="0.1524" layer="91"/>
-<label x="93.98" y="78.74" size="1.27" layer="95" rot="R180" xref="yes"/>
 </segment>
 </net>
@@
 <label x="195.58" y="142.24" size="1.27" layer="95" rot="R180" xref="yes"/>
 </segment>
+<segment>
+<pinref part="U1" gate="G$1" pin="P1.11"/>
+<wire x1="144.78" y1="101.6" x2="147.32" y2="101.6" width="0.1524" layer="91"/>
+<label x="147.32" y="101.6" size="1.27" layer="95" xref="yes"/>
+</segment>
 </net>
 <net name="N$41" class="0">
@@
 </segment>
 </net>
-<net name="ACC_CS" class="0">
-<segment>
-<pinref part="U1" gate="G$1" pin="P0.15"/>
-<wire x1="99.06" y1="88.9" x2="93.98" y2="88.9" width="0.1524" layer="91"/>
-<label x="93.98" y="88.9" size="1.27" layer="95" rot="R180" xref="yes"/>
-</segment>
-</net>
 <net name="VSEC" class="0">
 <segment>
@@
 <wire x1="152.4" y1="152.4" x2="152.4" y2="154.94" width="0.1524" layer="91"/>
 <pinref part="P+3" gate="G$1" pin="VSEC"/>
+</segment>
+</net>
+<net name="ACC_CS" class="0">
+<segment>
+<pinref part="U1" gate="G$1" pin="P0.13"/>
+<wire x1="99.06" y1="93.98" x2="93.98" y2="93.98" width="0.1524" layer="91"/>
+<label x="93.98" y="93.98" size="1.27" layer="95" rot="R180" xref="yes"/>
+</segment>
+</net>
+<net name="!CLR_EN" class="0">
+<segment>
+<pinref part="U1" gate="G$1" pin="P0.11"/>
+<wire x1="99.06" y1="99.06" x2="93.98" y2="99.06" width="0.1524" layer="91"/>
+<label x="93.98" y="99.06" size="1.27" layer="95" rot="R180" xref="yes"/>
+</segment>
+</net>
+<net name="!RTC_IRQ3" class="0">
+<segment>
+<pinref part="U1" gate="G$1" pin="P1.07"/>
+<wire x1="144.78" y1="111.76" x2="147.32" y2="111.76" width="0.1524" layer="91"/>
+<label x="147.32" y="111.76" size="1.27" layer="95" xref="yes"/>
+</segment>
+<segment>
+<pinref part="U9" gate="G$1" pin="CLKOUT/!IRQ3"/>
+<wire x1="83.82" y1="27.94" x2="86.36" y2="27.94" width="0.1524" layer="91"/>
+<label x="86.36" y="27.94" size="1.27" layer="95" xref="yes"/>
 </segment>
 </net>
@@
 </drawing>
 <compatibility>
+<note version="6.3" minversion="6.2.2" severity="warning">
+Since Version 6.2.2 text objects can contain more than one line,
+which will not be processed correctly with this version.
+</note>
 <note version="8.2" severity="warning">
 Since Version 8.2, EAGLE supports online libraries. The ids

Commit message: Rearrange a bit
Connections:
- removed net N$43: JP6.2, TP23.TESTPOINT
- net VBAT: now also JP6.2, TP23.TESTPOINT
Changed lines of the file:
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@@
 </segment>
 <segment>
+<pinref part="JP6" gate="A" pin="2"/>
+<wire x1="20.32" y1="45.72" x2="25.4" y2="45.72" width="0.1524" layer="91"/>
+<pinref part="TP23" gate="G$1" pin="TESTPOINT"/>
+<wire x1="25.4" y1="45.72" x2="38.1" y2="45.72" width="0.1524" layer="91"/>
+<junction x="25.4" y="45.72"/>
 <pinref part="P+13" gate="VCC" pin="VBAT"/>
 <wire x1="38.1" y1="48.26" x2="38.1" y2="45.72" width="0.1524" layer="91"/>
@@
 </segment>
 </net>
-<net name="N$43" class="0">
-<segment>
-<pinref part="JP6" gate="A" pin="2"/>
-<wire x1="20.32" y1="45.72" x2="25.4" y2="45.72" width="0.1524" layer="91"/>
-<pinref part="TP23" gate="G$1" pin="TESTPOINT"/>
-<wire x1="25.4" y1="45.72" x2="38.1" y2="45.72" width="0.1524" layer="91"/>
-<junction x="25.4" y="45.72"/>
-</segment>
-</net>
