File: hardware/permamote_eval/rev_b/permamote.brd (EAGLE design)
At the start: 79.4 x 89.5 mm, 137 parts, among them J1 TC2030-JLINK-L, J2 M10X2, J3 M04X2, Q1 PMDXB950UPEL, Q10 CSD22206W, Q11 CSD22206W, Q2 PMDXB950UPEL, Q3 PMDXB950UPEL, Q4 PMDXB950UPEL, Q5 PMDXB950UPEL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

Commit message: WIP reroute signals
Parts:
- removed Q11, Q9: CSD22206W, fets:DSBGA
- added C41: 0.1uF, passives:0402_CAP
- added J5: MICRO_USB_B_HIROSE_ZX62R-B-5P, connector:USB_MICRO_B-HIROSE-ZX62R-B-5P
- added U12: FT232RQ, ftdichip:QFN32
- BT2, BT3: value BAT-HLD-20XX-THRU -> BAT-HLD-002-THM; device batteries:BAT-HLD-20XX-THRU -> batteries:BAT-HLD-002-THM
- C17: device passives:0603_CAP -> passives:0402_CAP
- D1: value SOLARCELL -> SOLARCELLSCREW; device mote:SOLAR_HOLES -> permamote:PHEONIX-1935161
- Q10, Q7, Q8: value CSD22206W -> PMDXB950UPEL; device fets:DSBGA -> fets:XDFN-6
- moved L8 194.6 mm to (51.3, 78.4), turned to 270 degrees
- moved R16 193.3 mm to (66.3, 74.7), turned to 270 degrees
- moved R14 188.9 mm to (64.3, 74.7), turned to 90 degrees
- moved R13 188.4 mm to (66.3, 77.2), turned to 90 degrees
- moved R12 183.0 mm to (64.3, 77.2), turned to 270 degrees
- moved SJ1 181.8 mm to (64.3, 85.9)
- moved R10 176.6 mm to (62.2, 75.9), turned to 270 degrees
- moved R29 174.3 mm to (66.3, 80.5), turned to 270 degrees
- moved R28 169.0 mm to (64.3, 80.5), turned to 90 degrees
- moved R21 164.7 mm to (62.2, 81.8), turned to 90 degrees
- moved R15 164.2 mm to (66.3, 83.1), turned to 90 degrees
- moved R11 159.0 mm to (64.3, 83.1), turned to 270 degrees
- moved Q6 145.0 mm to (48.5, 84.3), turned to 90 degrees
- moved Q5 137.2 mm to (44.7, 84.3), turned to 90 degrees
- moved U2 134.4 mm to (54.1, 84.1), turned to 90 degrees
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Connections:
- net N$46 renamed !VBAT_SEC_ON
- net N$56 renamed !VBAT_PRI_ON
- removed net !ACC_EN: J2.15, U10.A14, U9.22
- removed net !I2C_EN: J2.3
- new net D+: J5.3, U12.14
- new net D-: J5.2, U12.15
- new net DBG_RX: J2.5, U10.R1, U12.30, U9.43
- new net DBG_TX: J2.7, U10.U1, U12.2, U9.44
- new net N$13: C41.1, U12.16
- new net USB_5V: J5.1, U12.19
- net !CLR_EN: now also J2.11, Q7.2; no longer J2.9, Q7.A1
- net !HUM_EN: now also Q8.5, U10.J24; no longer Q10.A1, U10.U1
- net !LT_EN: now also J2.13, Q7.5; no longer J2.11, Q8.A1
- net !PIR_EN: now also J2.15, Q10.2; no longer J2.13, Q11.A1
- net !PR_EN: now also J2.9, Q8.2; no longer J2.7, Q9.A1
- net !RST: now also U12.18
- net !RTC_IRQ1: no longer U9.44
- net !RTC_IRQ2: no longer U9.43
- net GND: now also C41.2, D1.2, J5.5, U12.17, U12.20, U12.24, U12.26, U12.4; no longer D1.-
- net MOSI: now also J2.3; no longer J2.5
- net N$19: now also Q8.1; no longer Q9.A2, Q9.A3, Q9.B1, Q9.B2, Q9.B3
- net N$20: now also Q7.3; no longer Q8.C1, Q8.C2, Q8.C3
- net N$21: now also Q8.6; no longer Q9.C1, Q9.C2, Q9.C3
- net N$22: now also Q8.3; no longer Q10.C1, Q10.C2, Q10.C3
- net N$23: now also Q10.6; no longer Q11.C1, Q11.C2, Q11.C3
- net N$24: now also Q10.1; no longer Q11.A2, Q11.A3, Q11.B1, Q11.B2, Q11.B3
- net N$31: now also Q7.6; no longer Q7.C1, Q7.C2, Q7.C3
- net N$33: now also Q7.1; no longer Q7.A2, Q7.A3, Q7.B1, Q7.B2, Q7.B3
- net N$36: now also Q8.4; no longer Q10.A2, Q10.A3, Q10.B1, Q10.B2, Q10.B3
- net N$37: now also Q7.4; no longer Q8.A2, Q8.A3, Q8.B1, Q8.B2, Q8.B3
- net VBAT: now also BT2.POS1, BT2.POS2, BT2.POS3, BT2.POS4, BT3.POS1, BT3.POS2, BT3.POS3, BT3.POS4; no longer BT2.+1, BT2.+2, BT2.+3, BT2.+4, BT3.+1, BT3.+2, BT3.+3, BT3.+4
- net VCC: now also U12.1
- net VSOL: now also D1.1; no longer D1.+
Routing:
- net !ACC_EN: track 98.5 -> 0.00 mm, vias 3 -> 0
- net VSOL: track 155.2 -> 76.1 mm
- net DBG_RX: track 0.00 -> 71.1 mm, vias 0 -> 4
- net DBG_TX: track 0.00 -> 70.1 mm, vias 0 -> 4
- net VBAT: track 219.8 -> 154.2 mm
- net !RST: track 160.4 -> 106.4 mm
- net SDA: track 181.7 -> 127.9 mm, vias 9 -> 10
- net !RTC_IRQ1: track 122.0 -> 71.6 mm, vias 7 -> 5
- net !RTC_IRQ2: track 126.2 -> 76.7 mm, vias 6 -> 5
- net SCK: track 155.9 -> 107.5 mm, vias 6 -> 7
- net SW: track 103.3 -> 55.0 mm, vias 5 -> 4
- net SCL: track 187.9 -> 139.7 mm
- net !LT_EN: track 143.7 -> 96.0 mm, vias 7 -> 6
- net PIR_OUT: track 138.5 -> 93.4 mm
- net VSEC: track 137.9 -> 95.3 mm, vias 3 -> 2
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- added copper zone on layer 1, net N$10
- added copper zone on layer 1, net N$11
- added copper zone on layer 1, net N$17
- added copper zone on layer 15, net VBAT
- added copper zone on layer 1, net VSOL
Other:
- board text added: "+"
- board text added: ">REV"
- board text removed: "2/3 AA"
- board text removed: "AA"
- board text removed: "CR123A"

Commit message: WIP route test signals + change rtc source
Parts:
- added JP17, JP18: (no value), SparkFun-Passives:SJ_2S
- added JP19: (no value), SparkFun-Connectors:1X02
- moved C41 236.1 mm to (44.8, 83.2), turned to 180 degrees
- moved J5 233.5 mm to (46.4, 89.3), turned to 180 degrees
- moved U12 216.5 mm to (47.3, 79.6), turned to 180 degrees
- moved TP10 38.7 mm to (68.2, 87.1)
- moved SJ1 20.4 mm to (66.2, 65.5), turned to 270 degrees
- moved Q5 20.0 mm to (64.6, 85.1), turned to 0 degrees
- moved R15 19.8 mm to (63.4, 63.5), turned to 0 degrees
- moved R29 17.9 mm to (60.8, 63.5), turned to 180 degrees
- moved C37 17.8 mm to (62.0, 85.2), turned to 90 degrees
- moved R11 17.5 mm to (63.4, 65.5), turned to 180 degrees
- moved R22 16.5 mm to (60.2, 85.2), turned to 90 degrees
- moved Q6 16.4 mm to (64.6, 81.3), turned to 0 degrees
- moved R13 16.3 mm to (57.5, 63.5), turned to 0 degrees
- moved R16 15.9 mm to (55.0, 63.5), turned to 180 degrees
- moved R9 15.7 mm to (58.8, 85.2), turned to 270 degrees
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Connections:
- new net N$46: JP17.1, U12.18
- new net N$56: JP18.1, JP19.1, U1.5
- net !RST: now also JP17.2; no longer U12.18
- net VBAT: now also JP18.2, JP19.2; no longer JP10.2, JP6.2, R6.2, R7.2
- net VCC: now also JP10.2, JP6.2, R6.2, R7.2
Routing:
- net DBG_TX: track 70.1 -> 153.6 mm, vias 4 -> 5
- net DBG_RX: track 71.1 -> 152.7 mm, vias 4 -> 5
- net !RST: track 106.4 -> 173.3 mm, vias 5 -> 6
- net SW: track 55.0 -> 117.9 mm, vias 4 -> 7
- net VSEC: track 95.3 -> 151.7 mm, vias 2 -> 3
- net SCK: track 107.5 -> 158.5 mm
- net N$56: track 0.00 -> 50.2 mm, vias 0 -> 1
- net !LT_EN: track 96.0 -> 145.8 mm
- net !CLR_EN: track 121.0 -> 169.7 mm
- net !PR_EN: track 104.5 -> 150.9 mm
- net VSOL: track 76.1 -> 122.0 mm, vias 5 -> 6
- net !LT_INT: track 128.0 -> 173.4 mm
- net SDA: track 127.9 -> 172.9 mm
- net PIR_OUT: track 93.4 -> 138.2 mm
- net !CLR_INT: track 121.8 -> 164.0 mm
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Other:
- board text added: "DBG_RX"
- board text added: "DBG_TX"
- board text added: "RTC BAT"
- board text removed: "!ACC_EN"
- board text removed: "!I2C_EN"

Commit message: Nothing to do - all airwires routed
Also fixed paste for NRF52840, attempted to fix keepout/stop layers for
pfet arrays
Parts:
- moved R3 12.9 mm to (27.9, 17.7)
- moved R2 12.2 mm to (25.9, 17.0)
- moved L1 0.13 mm to (7.37, 71.3)
- moved C1 0.13 mm to (6.10, 70.9)
Routing:
- net N$58: track 21.5 -> 26.1 mm
- net VCC: track 46.1 -> 41.7 mm, vias 5 -> 6
- net SCL: track 180.8 -> 176.5 mm, vias 10 -> 9
- net GND: track 49.7 -> 52.7 mm
- net !PIR_EN: track 118.8 -> 117.6 mm
- net SDA: track 172.9 -> 173.8 mm, vias 10 -> 9
- net N$19: track 27.8 -> 28.4 mm

Commit message: Rearrange some labels, notes
Note that i2c pullups do not need to be populated
Other:
- board text added: "L"
- board text added: "T"

Commit message: incorporate Branden's changes
Parts:
- added JP20, JP21, JP22: (no value), SparkFun-Passives:SJ_2S
- JP17: device SparkFun-Passives:SJ_2S -> SparkFun-Passives:SJ_2S-NO
- moved R5 4.86 mm to (13.2, 15.6), turned to 0 degrees
- moved R4 1.80 mm to (21.8, 16.8), turned to 180 degrees
- moved JP18 1.17 mm to (55.0, 37.0)
- moved JP19 1.17 mm to (58.0, 39.4)
Connections:
- net N$13 renamed 3V3OUT
- removed net N$20: Q7.3, U7.1
- new net N$13: JP22.2, U12.1
- new net N$59: Q7.3, R5.2, U7.1
- new net RXD: JP21.1, U12.2
- new net TXD: JP20.1, U12.30
- net DBG_RX: now also JP20.2; no longer U12.30
- net DBG_TX: now also JP21.2; no longer U12.2
- net N$31: now also R4.2
- net N$33: no longer R4.2
- net N$37: no longer R5.2
- net VCC: now also JP22.1; no longer U12.1
Routing:
- net N$59: track 0.00 -> 12.7 mm, vias 0 -> 2
- net N$20: track 9.20 -> 0.00 mm, vias 2 -> 0
- net N$31: track 7.24 -> 13.8 mm
- net RXD: track 0.00 -> 5.80 mm, vias 0 -> 2
- net N$13: track 0.00 -> 3.97 mm
- net TXD: track 0.00 -> 3.89 mm
- net DBG_RX: track 152.7 -> 149.7 mm
- net !LT_INT: track 173.4 -> 170.5 mm
- net DBG_TX: track 153.6 -> 151.0 mm
- net N$33: track 30.8 -> 28.5 mm
- net GND: track 52.7 -> 53.4 mm, vias 80 -> 82
- net VCC: track 41.7 -> 42.3 mm
- net N$37: track 17.2 -> 16.6 mm
- net !CLR_INT: track 164.0 -> 163.5 mm
Other:
- board text added: "FTDI Isolation"
- board text added: "Permamote Eval Neal Jackson 12/17"
- board text removed: "Permamote Eval Neal Jackson 10/17"

Commit message: add vanadium battery
Parts:
- added BT5: VL-2020, batteries:VL-2020
Connections:
- net GND: now also BT5.-
- net VSEC: now also BT5.+
Routing:
- net VSEC: track 151.7 -> 173.6 mm
- net SW: track 117.9 -> 118.5 mm
- net GND: vias 82 -> 111
Changed lines of the file:
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@@
 </element>
 <element name="D1" library="permamote" package="PHEONIX-1935161" value="SOLARCELLSCREW" x="74.168" y="60.198" smashed="yes" rot="R90">
-<attribute name="NAME" x="70.104" y="68.072" size="1.016" layer="25" font="vector" ratio="12"/>
+<attribute name="NAME" x="69.85" y="57.658" size="1.016" layer="25" font="vector" ratio="12" rot="R90"/>
 </element>
 <element name="JP17" library="SparkFun-Passives" package="SJ_2S-NO" value="" x="41.529" y="81.28" smashed="yes" rot="R180">
@@
 <element name="JP22" library="SparkFun-Passives" package="SJ_2S" value="" x="51.308" y="74.803" smashed="yes">
 <attribute name="VALUE" x="50.3582" y="73.152" size="0.4064" layer="27"/>
+</element>
+<element name="BT5" library="batteries" package="VL-2020" value="VL-2020" x="57.15" y="55.626" rot="R180">
+<attribute name="DIGIKEY" value="P082-ND" x="57.15" y="55.626" size="0.8128" layer="27" font="vector" ratio="12" rot="R180" display="off"/>
+<attribute name="MANUFACTURER" value="PANASONIC" x="57.15" y="55.626" size="0.8128" layer="27" font="vector" ratio="12" rot="R180" display="off"/>
+<attribute name="MPN" value="VL-2020/VCN" x="57.15" y="55.626" size="0.8128" layer="27" font="vector" ratio="12" rot="R180" display="off"/>
 </element>
 </elements>
@@
 <via x="50.927" y="82.931" extent="1-16" drill="0.2032"/>
 <via x="47.879" y="82.931" extent="1-16" drill="0.2032"/>
+<contactref element="BT5" pad="-"/>
+<via x="5.08" y="73.279" extent="1-16" drill="0.2032"/>
+<via x="4.318" y="73.279" extent="1-16" drill="0.2032"/>
+<via x="3.556" y="73.279" extent="1-16" drill="0.2032"/>
+<via x="2.794" y="73.279" extent="1-16" drill="0.2032"/>
+<via x="2.032" y="73.279" extent="1-16" drill="0.2032"/>
+<via x="1.27" y="73.279" extent="1-16" drill="0.2032"/>
+<via x="0.508" y="73.279" extent="1-16" drill="0.2032"/>
+<via x="5.08" y="67.437" extent="1-16" drill="0.2032"/>
+<via x="4.318" y="67.437" extent="1-16" drill="0.2032"/>
+<via x="3.556" y="67.437" extent="1-16" drill="0.2032"/>
+<via x="2.794" y="67.437" extent="1-16" drill="0.2032"/>
+<via x="2.032" y="67.437" extent="1-16" drill="0.2032"/>
+<via x="1.27" y="67.437" extent="1-16" drill="0.2032"/>
+<via x="0.508" y="67.437" extent="1-16" drill="0.2032"/>
+<via x="7.493" y="46.736" extent="1-16" drill="0.2032"/>
+<via x="5.842" y="52.07" extent="1-16" drill="0.2032"/>
+<via x="5.08" y="52.07" extent="1-16" drill="0.2032"/>
+<via x="4.318" y="52.07" extent="1-16" drill="0.2032"/>
+<via x="3.429" y="52.07" extent="1-16" drill="0.2032"/>
+<via x="2.667" y="52.07" extent="1-16" drill="0.2032"/>
+<via x="1.905" y="52.07" extent="1-16" drill="0.2032"/>
+<via x="1.143" y="52.07" extent="1-16" drill="0.2032"/>
+<via x="5.715" y="57.912" extent="1-16" drill="0.2032"/>
+<via x="4.953" y="57.912" extent="1-16" drill="0.2032"/>
+<via x="4.191" y="57.912" extent="1-16" drill="0.2032"/>
+<via x="3.429" y="57.912" extent="1-16" drill="0.2032"/>
+<via x="2.667" y="57.912" extent="1-16" drill="0.2032"/>
+<via x="1.905" y="57.912" extent="1-16" drill="0.2032"/>
+<via x="1.143" y="57.912" extent="1-16" drill="0.2032"/>
+<wire x1="0.381" y1="57.912" x2="0.381" y2="57.912" width="0" layer="19" extent="1-16"/>
+<wire x1="0.381" y1="52.07" x2="0.381" y2="52.07" width="0" layer="19" extent="1-16"/>
+<wire x1="6.42493125" y1="58.039" x2="5.715" y2="57.912" width="0" layer="19" extent="1-1"/>
+<wire x1="4.953" y1="57.912" x2="5.715" y2="57.912" width="0" layer="19" extent="1-1"/>
+<wire x1="4.191" y1="57.912" x2="4.953" y2="57.912" width="0" layer="19" extent="1-1"/>
+<wire x1="3.429" y1="57.912" x2="4.191" y2="57.912" width="0" layer="19" extent="1-1"/>
+<wire x1="2.667" y1="57.912" x2="3.429" y2="57.912" width="0" layer="19" extent="1-1"/>
+<wire x1="1.905" y1="57.912" x2="2.667" y2="57.912" width="0" layer="19" extent="1-1"/>
+<wire x1="1.143" y1="57.912" x2="1.905" y2="57.912" width="0" layer="19" extent="1-1"/>
+<wire x1="0.381" y1="57.912" x2="1.143" y2="57.912" width="0" layer="19" extent="1-1"/>
+<wire x1="5.842" y1="52.07" x2="6.858" y2="50.87493125" width="0" layer="19" extent="1-1"/>
+<wire x1="5.08" y1="52.07" x2="5.842" y2="52.07" width="0" layer="19" extent="1-1"/>
+<wire x1="4.318" y1="52.07" x2="5.08" y2="52.07" width="0" layer="19" extent="1-1"/>
+<wire x1="3.429" y1="52.07" x2="4.318" y2="52.07" width="0" layer="19" extent="1-1"/>
+<wire x1="2.667" y1="52.07" x2="3.429" y2="52.07" width="0" layer="19" extent="1-1"/>
+<wire x1="1.905" y1="52.07" x2="2.667" y2="52.07" width="0" layer="19" extent="1-1"/>
+<wire x1="1.143" y1="52.07" x2="1.905" y2="52.07" width="0" layer="19" extent="1-1"/>
+<wire x1="0.381" y1="52.07" x2="1.143" y2="52.07" width="0" layer="19" extent="1-1"/>
+<wire x1="1.524" y1="53.285" x2="1.905" y2="52.07" width="0" layer="19" extent="1-1"/>
+<wire x1="7.493" y1="46.736" x2="6.858" y2="50.87493125" width="0" layer="19" extent="1-1"/>
 </signal>
 <signal name="N$8">
@@
 <wire x1="58.039" y1="36.83" x2="49.149" y2="36.83" width="0.254" layer="15"/>
 <wire x1="49.149" y1="36.83" x2="48.26" y2="35.941" width="0.254" layer="15"/>
-<wire x1="70.09" y1="8.56" x2="70.09" y2="11.66" width="0" layer="19" extent="1-1"/>
-<wire x1="49.29" y1="11.66" x2="70.09" y2="11.66" width="0" layer="19" extent="1-1"/>
-<wire x1="48.26" y1="10.033" x2="49.29" y2="11.66" width="0" layer="19" extent="1-15"/>
-<wire x1="49.29" y1="8.56" x2="48.26" y2="10.033" width="0" layer="19" extent="1-15"/>
-<wire x1="47.23" y1="8.56" x2="48.26" y2="10.033" width="0" layer="19" extent="1-15"/>
-<wire x1="47.23" y1="11.66" x2="48.26" y2="10.033" width="0" layer="19" extent="1-15"/>
-<wire x1="26.43" y1="11.66" x2="47.23" y2="11.66" width="0" layer="19" extent="1-1"/>
-<wire x1="26.43" y1="8.56" x2="26.43" y2="11.66" width="0" layer="19" extent="1-1"/>
 </signal>
 <signal name="N$15">
@@
 <wire x1="35.306" y1="73.66" x2="41.275" y2="73.66" width="0.254" layer="16"/>
 <wire x1="41.275" y1="73.66" x2="48.387" y2="80.772" width="0.254" layer="16"/>
-<wire x1="72.136" y1="49.403" x2="62.103" y2="59.436" width="0.254" layer="1"/>
-<wire x1="62.103" y1="59.436" x2="55.499" y2="59.436" width="0.254" layer="1"/>
+<wire x1="62.103" y1="59.436" x2="61.976" y2="59.436" width="0.254" layer="1"/>
 <via x="55.499" y="59.436" extent="1-16" drill="0.2032"/>
+<wire x1="61.976" y1="59.436" x2="55.499" y2="59.436" width="0.254" layer="1"/>
 <wire x1="55.499" y1="59.436" x2="54.483" y2="60.452" width="0.254" layer="15"/>
 <wire x1="54.483" y1="60.452" x2="54.483" y2="76.073" width="0.254" layer="15"/>
@@
 <wire x1="54.483" y1="76.073" x2="56.261" y2="77.851" width="0.254" layer="1"/>
 <wire x1="56.261" y1="77.851" x2="56.261" y2="78.359" width="0.254" layer="1"/>
+<wire x1="61.976" y1="59.436" x2="62.865" y2="59.436" width="0.254" layer="1"/>
+<wire x1="62.865" y1="59.436" x2="72.136" y2="50.165" width="0.254" layer="1"/>
+<wire x1="72.136" y1="50.165" x2="72.136" y2="49.403" width="0.254" layer="1"/>
 </signal>
 <signal name="!LT_EN">
@@
 <wire x1="60.833" y1="75.692" x2="62.649" y2="75.692" width="0.254" layer="1"/>
 <wire x1="55.499" y1="60.452" x2="65.024" y2="60.452" width="0.8128" layer="1"/>
-<wire x1="71.287" y1="66.715" x2="71.287" y2="75.184" width="0.8128" layer="1"/>
+<wire x1="71.287" y1="70.104" x2="71.287" y2="66.715" width="0.8128" layer="1"/>
+<wire x1="71.287" y1="70.104" x2="71.287" y2="75.184" width="0.8128" layer="1"/>
 <wire x1="70.5485" y1="65.9765" x2="65.024" y2="60.452" width="0.8128" layer="1"/>
 <wire x1="70.5485" y1="65.9765" x2="71.287" y2="66.715" width="0.8128" layer="1"/>
@@
 <wire x1="76.454" y1="60.071" x2="70.5485" y2="65.9765" width="0.254" layer="1"/>
 <wire x1="76.454" y1="48.641" x2="76.454" y2="60.071" width="0.254" layer="1"/>
+<contactref element="BT5" pad="+"/>
+<wire x1="71.307" y1="70.084" x2="71.287" y2="70.104" width="0.8128" layer="1"/>
+<wire x1="62.25" y1="56.976" x2="71.287" y2="66.013" width="0.8128" layer="15"/>
+<wire x1="71.287" y1="66.013" x2="71.287" y2="75.184" width="0.8128" layer="15"/>
 </signal>
 <signal name="!CLR_EN">
@@
 <wire x1="22.987" y1="79.883" x2="24.15320625" y2="79.883" width="0.1016" layer="1"/>
 </signal>
-<signal name="N$28">
-<via x="7.493" y="46.736" extent="1-16" drill="0.2032"/>
-</signal>
 <signal name="N$29">
