File: hardware/permamote/rev_a/permamote.brd (EAGLE design)
At the start: 27 x 60.1 mm, 131 parts, among them J1 TC2030-JLINK-NL, J5 MICRO_USB_B_HIROSE_ZX62R-B-5P, Q1 PMDXB950UPEL, Q10 PMDXB950UPEL, Q2 PMDXB950UPEL, Q3 PMDXB950UPEL, Q4 PMDXB950UPEL, Q5 PMDXB950UPEL, Q6 PMDXB950UPEL, Q7 PMDXB950UPEL, Q8 PMDXB950UPEL, U1 AB1815-T3, U10 NRF52840, U11 SI7021-A20-GM1, U2 BQ25505, U3 EKMB1101111, U4 FT232RQ, U5 ISL29125, U6 LIS2DW12, U7 MAX17222, U8 MAX44009, U9 MS5637-02BA03, X1 32MHz, X3 32.768kHz, X4 ABS07-32.768KHZ-7-T

Commit message: update parts
Parts:
- C28: device passives:0603_CAP -> passives:0402_CAP
- J5: value MICRO_USB_B_HIROSE_ZX62R-B-5P -> MICRO_USB_B_HIROSE_ZX62R-B-5P(30); device connector:USB_MICRO_B-HIROSE-ZX62R-B-5P -> connector:MICRO_USB_B_HIROSE_ZX62R-B-5P(30)
- R15: value 4.22M -> DNP
- R16: value 5.62M -> DNP
- R17: value 6.19M -> 6.2M
- R18: value 6.81M -> 6.8M
- R19: value 7.32M -> DNP
- R20: value 8.87M -> DNP
- R21: value 9.09M -> 9.1M
- R5: value 6.04k -> DNP
Changed lines of the file:
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@@
 </element>
 <element name="R14" library="passives" package="0402_RES" value="3.9M" x="12.192" y="57.404" smashed="yes" rot="R270">
-<attribute name="DIGIKEY" value="YAG3306CT-ND" x="12.192" y="57.404" size="1.778" layer="27" font="vector" ratio="12" rot="R270" display="off"/>
+<attribute name="DIGIKEY" value="YAG3301CT-ND" x="12.192" y="57.404" size="1.778" layer="27" font="vector" ratio="12" rot="R270" display="off"/>
+<attribute name="MPN" value="RC0402JR-073M9L" x="12.192" y="57.404" size="1.778" layer="27" rot="R270" display="off"/>
 <attribute name="NAME" x="12.192" y="58.42" size="1.016" layer="25" font="vector" ratio="12" align="bottom-center"/>
 <attribute name="VALUE" x="10.795" y="57.404" size="1.016" layer="27" font="vector" ratio="12" rot="R270" align="bottom-center"/>
 </element>
-<element name="R21" library="passives" package="0402_RES" value="9.09M" x="13.716" y="57.404" smashed="yes" rot="R90">
-<attribute name="DIGIKEY" value="YAG3306CT-ND" x="13.716" y="57.404" size="1.778" layer="27" font="vector" ratio="12" rot="R90" display="off"/>
+<element name="R21" library="passives" package="0402_RES" value="9.1M" x="13.716" y="57.404" smashed="yes" rot="R90">
+<attribute name="DIGIKEY" value="YAG3322CT-ND" x="13.716" y="57.404" size="1.778" layer="27" font="vector" ratio="12" rot="R90" display="off"/>
+<attribute name="MPN" value="RC0402JR-079M1L" x="13.716" y="57.404" size="1.778" layer="27" rot="R90" display="off"/>
 <attribute name="NAME" x="15.24" y="58.42" size="1.016" layer="25" font="vector" ratio="12" rot="R90" align="bottom-center"/>
 <attribute name="VALUE" x="15.113" y="57.404" size="1.016" layer="27" font="vector" ratio="12" rot="R90" align="bottom-center"/>
 </element>
 <element name="R4" library="passives" package="0402_RES" value="6.04k" x="11.176" y="56.388" smashed="yes" rot="R90">
-<attribute name="DIGIKEY" value="YAG3306CT-ND" x="11.176" y="56.388" size="1.778" layer="27" font="vector" ratio="12" rot="R90" display="off"/>
+<attribute name="DIGIKEY" value="YAG2293CT-ND" x="11.176" y="56.388" size="1.778" layer="27" font="vector" ratio="12" rot="R90" display="off"/>
+<attribute name="MPN" value="RC0402FR-076K04L" x="11.176" y="56.388" size="1.778" layer="27" rot="R90" display="off"/>
 <attribute name="NAME" x="10.795" y="56.896" size="1.016" layer="25" font="vector" ratio="12" rot="R90" align="bottom-center"/>
 <attribute name="VALUE" x="12.573" y="56.388" size="1.016" layer="27" font="vector" ratio="12" rot="R90" align="bottom-center"/>
 </element>
-<element name="R17" library="passives" package="0402_RES" value="6.19M" x="12.192" y="55.372" smashed="yes" rot="R90">
-<attribute name="DIGIKEY" value="YAG3306CT-ND" x="12.192" y="55.372" size="1.778" layer="27" font="vector" ratio="12" rot="R90" display="off"/>
+<element name="R17" library="passives" package="0402_RES" value="6.2M" x="12.192" y="55.372" smashed="yes" rot="R90">
+<attribute name="DIGIKEY" value="YAG3309CT-ND" x="12.192" y="55.372" size="1.778" layer="27" font="vector" ratio="12" rot="R90" display="off"/>
+<attribute name="MPN" value="RC0402JR-076M2L" x="12.192" y="55.372" size="1.778" layer="27" rot="R90" display="off"/>
 <attribute name="NAME" x="10.541" y="55.245" size="1.016" layer="25" font="vector" ratio="12" rot="R180" align="bottom-center"/>
 <attribute name="VALUE" x="13.589" y="55.372" size="1.016" layer="27" font="vector" ratio="12" rot="R90" align="bottom-center"/>
 </element>
-<element name="R18" library="passives" package="0402_RES" value="6.81M" x="13.716" y="55.372" smashed="yes" rot="R270">
-<attribute name="DIGIKEY" value="YAG3306CT-ND" x="13.716" y="55.372" size="1.778" layer="27" font="vector" ratio="12" rot="R270" display="off"/>
+<element name="R18" library="passives" package="0402_RES" value="6.8M" x="13.716" y="55.372" smashed="yes" rot="R270">
+<attribute name="DIGIKEY" value="YAG3310CT-ND" x="13.716" y="55.372" size="1.778" layer="27" font="vector" ratio="12" rot="R270" display="off"/>
+<attribute name="MPN" value="RC0402JR-076M8L" x="13.716" y="55.372" size="1.778" layer="27" rot="R270" display="off"/>
 <attribute name="NAME" x="14.097" y="55.372" size="1.016" layer="25" font="vector" ratio="12" rot="R270" align="bottom-center"/>
 <attribute name="VALUE" x="12.319" y="55.372" size="1.016" layer="27" font="vector" ratio="12" rot="R270" align="bottom-center"/>
@@
 <attribute name="VALUE" x="20.0929" y="57.626" size="0.02" layer="27"/>
 </element>
-<element name="R5" library="passives" package="0402_RES" value="6.04k" x="10.414" y="51.816" smashed="yes" rot="R270">
+<element name="R5" library="passives" package="0402_RES" value="DNP" x="10.414" y="51.816" smashed="yes" rot="R270">
 <attribute name="DIGIKEY" value="YAG3306CT-ND" x="10.414" y="51.816" size="1.778" layer="27" font="vector" ratio="12" rot="R270" display="off"/>
 <attribute name="NAME" x="10.033" y="51.308" size="1.016" layer="25" font="vector" ratio="12" rot="R90" align="bottom-center"/>
 <attribute name="VALUE" x="9.017" y="51.816" size="1.016" layer="27" font="vector" ratio="12" rot="R270" align="bottom-center"/>
 </element>
-<element name="R20" library="passives" package="0402_RES" value="8.87M" x="11.43" y="52.832" smashed="yes" rot="R270">
+<element name="R20" library="passives" package="0402_RES" value="DNP" x="11.43" y="52.832" smashed="yes" rot="R270">
 <attribute name="DIGIKEY" value="YAG3306CT-ND" x="11.43" y="52.832" size="1.778" layer="27" font="vector" ratio="12" rot="R270" display="off"/>
 <attribute name="NAME" x="9.779" y="53.594" size="1.016" layer="25" font="vector" ratio="12" rot="R180" align="bottom-center"/>
 <attribute name="VALUE" x="10.033" y="52.832" size="1.016" layer="27" font="vector" ratio="12" rot="R270" align="bottom-center"/>
 </element>
-<element name="R15" library="passives" package="0402_RES" value="4.22M" x="12.7" y="52.832" smashed="yes" rot="R90">
+<element name="R15" library="passives" package="0402_RES" value="DNP" x="12.7" y="52.832" smashed="yes" rot="R90">
 <attribute name="DIGIKEY" value="YAG3306CT-ND" x="12.7" y="52.832" size="1.778" layer="27" font="vector" ratio="12" rot="R90" display="off"/>
 <attribute name="NAME" x="14.224" y="52.324" size="1.016" layer="25" font="vector" ratio="12" align="bottom-center"/>
@@
 <attribute name="NAME" x="21.803" y="38.1" size="1.016" layer="26" font="vector" ratio="12" rot="MR90" align="bottom-center"/>
 </element>
-<element name="R19" library="passives" package="0402_RES" value="7.32M" x="11.43" y="50.8" smashed="yes" rot="R90">
+<element name="R19" library="passives" package="0402_RES" value="DNP" x="11.43" y="50.8" smashed="yes" rot="R90">
 <attribute name="DIGIKEY" value="YAG3306CT-ND" x="11.43" y="50.8" size="1.778" layer="27" font="vector" ratio="12" rot="R90" display="off"/>
 <attribute name="NAME" x="11.43" y="49.911" size="1.016" layer="25" font="vector" ratio="12" rot="R180" align="bottom-center"/>
 <attribute name="VALUE" x="12.827" y="50.8" size="1.016" layer="27" font="vector" ratio="12" rot="R90" align="bottom-center"/>
 </element>
-<element name="R16" library="passives" package="0402_RES" value="5.62M" x="12.7" y="50.8" smashed="yes" rot="R270">
+<element name="R16" library="passives" package="0402_RES" value="DNP" x="12.7" y="50.8" smashed="yes" rot="R270">
 <attribute name="DIGIKEY" value="YAG3306CT-ND" x="12.7" y="50.8" size="1.778" layer="27" font="vector" ratio="12" rot="R270" display="off"/>
 <attribute name="NAME" x="13.081" y="50.8" size="1.016" layer="25" font="vector" ratio="12" rot="R270" align="bottom-center"/>
@@
 <attribute name="VALUE" x="2.286" y="28.956" size="1.016" layer="27" font="vector" ratio="12" rot="R90" align="bottom-center"/>
 </element>
-<element name="J5" library="connector" package="USB_MICRO_B-HIROSE-ZX62R-B-5P" value="MICRO_USB_B_HIROSE_ZX62R-B-5P" x="5.5" y="60" smashed="yes" rot="R180">
-<attribute name="DIGIKEY" value="H11574CT-ND" x="5.5" y="60" size="1.778" layer="27" rot="R180" display="off"/>
-<attribute name="MOUSER" value="798-ZX62R-B-5P" x="5.5" y="60" size="1.778" layer="27" rot="R180" display="off"/>
+<element name="J5" library="connector" package="MICRO_USB_B_HIROSE_ZX62R-B-5P(30)" value="MICRO_USB_B_HIROSE_ZX62R-B-5P(30)" x="5.5" y="60" smashed="yes" rot="R180">
+<attribute name="DIGIKEY" value="H125274CT-ND" x="5.5" y="60" size="1.778" layer="27" rot="R180" display="off"/>
+<attribute name="MOUSER" value="798-ZX62R-B-5P30" x="5.5" y="60" size="1.778" layer="27" rot="R180" display="off"/>
+<attribute name="MPN" value="ZX62R-B-5P(30)" x="5.5" y="60" size="1.778" layer="27" rot="R180" display="off"/>
 <attribute name="NAME" x="5.5" y="54.9" size="1.016" layer="25" font="vector" ratio="12" rot="R180" align="bottom-center"/>
-<attribute name="NEWARK" value="69W0714" x="5.5" y="60" size="1.778" layer="27" rot="R180" display="off"/>
+<attribute name="NEWARK" value="84Y6712" x="5.5" y="60" size="1.778" layer="27" rot="R180" display="off"/>
 <attribute name="VALUE" x="5.5" y="61.9" size="1.016" layer="27" font="vector" ratio="12" rot="R180" align="bottom-center"/>
 </element>
@@
 <attribute name="NAME" x="17.907" y="49.276" size="1.016" layer="25" font="vector" ratio="12" rot="R90" align="bottom-center"/>
 </element>
-<element name="C28" library="passives" package="0603_CAP" value="4.7uF" x="25.146" y="53.054" smashed="yes">
+<element name="C28" library="passives" package="0402_CAP" value="4.7uF" x="25.146" y="53.054" smashed="yes">
 <attribute name="DIGIKEY" value="445-5947-1-ND" x="25.146" y="53.054" size="1.778" layer="27" display="off"/>
 <attribute name="NAME" x="25.146" y="53.689" size="1.016" layer="25" font="vector" ratio="12" align="bottom-center"/>
