File: hardware/permamote/rev_a/permamote.sch (EAGLE design)
At the start: 130 parts, among them J1 TC2030-JLINK-NL, J5 MICRO_USB_B_HIROSE_ZX62R-B-5P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, Q1 PMDXB950UPEL, Q10 PMDXB950UPEL, Q2 PMDXB950UPEL, Q3 PMDXB950UPEL, Q4 PMDXB950UPEL, Q5 PMDXB950UPEL, Q6 PMDXB950UPEL, Q7 PMDXB950UPEL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

Commit message: Change attributes to include MPN, fix up BOM
Parts:
- BT2, BT3: DIGIKEY (none) -> BAT-HLD-001-THM-ND; MOUSER (none) -> 712-BAT-HLD-001-THM; MPN (none) -> BAT-HLD-001-THM
- C1: MPN (none) -> GRM1555C1HR50WA01D
- C10, C9: MPN (none) -> GRM155R71H103KA88D
- C11: MPN (none) -> C1005X7R1C473K050BC
- C12, C13, C14, C15, C16, C17, C18, C19, C20: MPN (none) -> GRM155R71C104KA88J
- C2: MPN (none) -> GRM1555C1HR80BA01D
- C21, C22, C23, C24, C25: MPN (none) -> GRM155R70G105KA12D
- C26, C27, C28: MPN (none) -> C1005X5R0J475K050BC
- C29, C30, C31: MPN (none) -> GRM188R60J106ME47D
- C3, C4, C5, C6: MPN (none) -> GRM1555C1H120GA01D
- C7: MPN (none) -> GRM1555C1H470JA01D
- C8: MPN (none) -> GRM1555C1H101JA01D
- L1: MPN (none) -> AISC-0402-3N3J-T
- L2: MPN (none) -> HK100515NJ-T
- L4: MPN (none) -> LQM18FN100M00D
- L5: MPN (none) -> 74437324220
- R1, R2, R3: MPN (none) -> RC0402JR-07470RL
- R10, R11, R12, R6, R7, R8, R9: MPN (none) -> RC0402JR-0710KL
- R13: MPN (none) -> RC0603FR-0780K6L
- R22: MPN (none) -> HMC0603JT33M0
- R23, R24, R25, R26, R27: MPN (none) -> HMC0402JT100M
- S1: MPN (none) -> EVQ-P2K02Q
- U11: MPN (none) -> SI7021-A20-GM1

Commit message: Fix NRF52840 via drill size
Update BOM
Parts:
- R6, R8: MPN RC0402JR-0710KL -> RC0402JR-0710KL
Changed lines of the file:
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@@
 <part name="R6" library="passives" deviceset="RESISTOR" device="0402_RES" value="10k">
 <attribute name="DIGIKEY" value="311-10KJRCT-ND "/>
-<attribute name="MPN" value="RC0402JR-0710KL "/>
+<attribute name="MPN" value="RC0402JR-0710KL"/>
 </part>
 <part name="P+8" library="supply1" library_urn="urn:adsk.eagle:library:371" deviceset="VCC" device=""/>
@@
 <part name="GND15" library="supply1" library_urn="urn:adsk.eagle:library:371" deviceset="GND" device=""/>
 <part name="U11" library="chips" deviceset="SI7021" device="-A20-GM1">
-<attribute name="MPN" value="SI7021-A20-GM1
-"/>
+<attribute name="MPN" value="SI7021-A20-GM1 "/>
 </part>
 <part name="C19" library="passives" deviceset="CAPACITOR" device="0402_CAP" value="0.1uF">
@@
 <part name="R8" library="passives" deviceset="RESISTOR" device="0402_RES" value="10k">
 <attribute name="DIGIKEY" value="311-10KJRCT-ND "/>
-<attribute name="MPN" value="RC0402JR-0710KL "/>
+<attribute name="MPN" value="RC0402JR-0710KL"/>
 </part>
 <part name="R9" library="passives" deviceset="RESISTOR" device="0402_RES" value="10k">
@@
 <part name="GND30" library="supply1" library_urn="urn:adsk.eagle:library:371" deviceset="GND" device=""/>
 <part name="S1" library="switches" deviceset="EVQP2" device="">
-<attribute name="MPN" value="EVQ-P2K02Q
-"/>
+<attribute name="MPN" value="EVQ-P2K02Q "/>
 </part>
 <part name="R10" library="passives" deviceset="RESISTOR" device="0402_RES" value="10k">
