File: hardware/permamote/rev_c/permamote.brd (EAGLE design)
At the start: 27 x 60 mm, 126 parts, among them J1 TC2030-JLINK-NL, J5 MICRO_USB_B_HIROSE_ZX62R-B-5P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, Q1 PMDXB950UPEL, Q10 PMDXB950UPEL, Q2 PMDXB950UPEL, Q3 PMDXB950UPEL, Q4 PMDXB950UPEL, Q5 PMDXB950UPEL, Q6 PMDXB950UPEL, Q7 PMDXB950UPEL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

Commit message: Change button, fixes #4
Parts:
- S1: value EVQP2 -> B3U-1000P; device switches:EVQP2 -> switches:B3U-1000P
- moved R2 5.01 mm to (11.4, 56.3)
- moved R1 4.33 mm to (12.7, 56.3)
- moved S1 3.89 mm to (15.5, 58.7), turned to 180 degrees
- moved D2 3.45 mm to (11.7, 58.5)
- moved R3 2.80 mm to (12.7, 53.7)
- moved J1 0.25 mm to (24.9, 30.9), flipped to the top
Connections:
- net !RTC_EXTR: now also S1.2; no longer S1.P$2, S1.P$4
- net GND: now also S1.1; no longer S1.P$1, S1.P$3
Routing:
- net N$15: track 10.8 -> 2.53 mm
- net N$17: track 8.82 -> 1.49 mm
- net LED_GREEN: track 50.5 -> 55.8 mm
- net N$19: track 8.60 -> 4.20 mm
- net LED_RED: track 50.0 -> 53.8 mm
- net LED_BLUE: track 50.7 -> 54.0 mm
- net SWDCLK: track 19.0 -> 15.7 mm, vias 3 -> 2
- net SWDIO: track 17.0 -> 13.6 mm, vias 3 -> 2
- net VCC: track 66.2 -> 67.3 mm
- net !RTC_EXTR: track 42.5 -> 41.6 mm, vias 4 -> 2
- net !RST: track 64.9 -> 65.5 mm, vias 4 -> 5
- net GND: vias 117 -> 110
Other:
- board text added: ">REV"
- board text added: "Permamote Neal Jackson 9/18"
- board text removed: "B"
- board text removed: "Permamote Neal Jackson 7/18"
