File: hardware/permacam/rev_a/permacam.sch (EAGLE design)
At the start: 110 parts, among them J1 TC2030-JLINK-NL, Q1 PMDXB950UPEL, Q2 PMDXB950UPEL, Q3 PMDXB950UPEL, Q4 PMDXB950UPEL, Q5 PMDXB950UPEL, Q6 PMDXB950UPEL, U1 AB1815-T3, U10 NRF52840, U2 BQ25505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

Commit message: Fix BOM errors for resistor + battery
Parts:
- BT2: DIGIKEY BAT-HLD-001-THM-ND -> (none); MPN BAT-HLD-001-THM -> (none)
- R10: DIGIKEY YAG3055CT-ND -> 311-215KHRCT-ND; MPN RC0402FR-07215KL -> RC0603FR-07215KL
Changed lines of the file:
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@@
 </part>
 <part name="R10" library="passives" deviceset="RESISTOR" device="0603_RES" value="215k">
-<attribute name="DIGIKEY" value="YAG3055CT-ND"/>
-<attribute name="MPN" value="RC0402FR-07215KL"/>
+<attribute name="DIGIKEY" value="311-215KHRCT-ND"/>
+<attribute name="MPN" value="RC0603FR-07215KL"/>
 </part>
 <part name="GND8" library="supply1" library_urn="urn:adsk.eagle:library:371" deviceset="GND" device=""/>
@@
 <part name="GND23" library="supply1" library_urn="urn:adsk.eagle:library:371" deviceset="GND" device=""/>
 <part name="GND19" library="supply1" library_urn="urn:adsk.eagle:library:371" deviceset="GND" device=""/>
-<part name="BT2" library="batteries" deviceset="2477THMCOINCELLCLIP" device="">
-<attribute name="DIGIKEY" value="BAT-HLD-001-THM-ND"/>
-<attribute name="MPN" value="BAT-HLD-001-THM"/>
-</part>
+<part name="BT2" library="batteries" deviceset="2477THMCOINCELLCLIP" device=""/>
 <part name="L3" library="passives" deviceset="INDUCTOR" device="IHL" value="1uH">
 <attribute name="DIGIKEY" value="541-1319-1-ND"/>
