File: hardware/permamote_lte/rev_a/permamote-lte.sch (EAGLE design)
At the start: 115 parts, among them J1 TC2030-JLINK-NL, J2 U.FL-R-SMT, J3 NANO_SIM, J4 U.FL-R-SMT, J5 DM3AT-SF-PEJM5, Q1 PMDXB950UPEL, Q10 PMDXB950UPEL, Q2 PMDXB950UPEL, Q3 PMDXB950UPEL, Q4 PMDXB950UPEL, Q5 PMDXB950UPEL, Q6 PMDXB950UPEL, Q7 PMDXB950UPEL, Q8 PMDXB950UPEL, U1 AB1815-T3, U10 SIP32510, U11 SI7021-A20-GM1, U12 TCS34725, U13 TPD3F303DPVR, U2 BQ25505, U3 EKMB1101111, U4 BGA725L6, U5 NRF9160, U6 LIS2DW12, U7 MAX17222, U8 MAX44009, U9 MS5637-02BA03, X4 ABS07-32.768KHZ-7-T

Commit message: fixes
Parts:
- L1: DIGIKEY (none) -> 490-2613-1-ND; MPN (none) -> LQG15HS1N8S02D
- L2: DIGIKEY (none) -> 490-6564-1-ND; MPN (none) -> LQG15HN5N1S02D
- L3: DIGIKEY (none) -> 490-6565-1-ND; MPN (none) -> LQG15HN7N5J02D
Changed lines of the file:
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@@
 <part name="GND2" library="supply1" library_urn="urn:adsk.eagle:library:371" deviceset="GND" device=""/>
 <part name="P+8" library="supply1" library_urn="urn:adsk.eagle:library:371" deviceset="VCC" device=""/>
-<part name="L3" library="passives" deviceset="INDUCTOR" device="0402" value="7.5nH"/>
+<part name="L3" library="passives" deviceset="INDUCTOR" device="0402" value="7.5nH">
+<attribute name="DIGIKEY" value="490-6565-1-ND"/>
+<attribute name="MPN" value="LQG15HN7N5J02D"/>
+</part>
 <part name="J4" library="connector" deviceset="U.FL-R-SMT" device=""/>
 <part name="GND28" library="supply1" library_urn="urn:adsk.eagle:library:371" deviceset="GND" device=""/>
@@
 <part name="GND33" library="supply1" library_urn="urn:adsk.eagle:library:371" deviceset="GND" device=""/>
 <part name="U4" library="chips" deviceset="BGA725L6" device=""/>
-<part name="L2" library="passives" deviceset="INDUCTOR" device="0402" value="5.1nH"/>
-<part name="L1" library="passives" deviceset="INDUCTOR" device="0402" value="1.8nH"/>
+<part name="L2" library="passives" deviceset="INDUCTOR" device="0402" value="5.1nH">
+<attribute name="DIGIKEY" value="490-6564-1-ND"/>
+<attribute name="MPN" value="LQG15HN5N1S02D"/>
+</part>
+<part name="L1" library="passives" deviceset="INDUCTOR" device="0402" value="1.8nH">
+<attribute name="DIGIKEY" value="490-2613-1-ND"/>
+<attribute name="MPN" value="LQG15HS1N8S02D"/>
+</part>
 <part name="C16" library="passives" deviceset="CAPACITOR" device="0402_CAP" value="4.7uF">
 <attribute name="DESCRIPTION" value="CAP CER 4.7UF 10V X5R 0402"/>
@@
 <attribute name="NAME" x="193.04" y="149.352" size="1.778" layer="95" ratio="12" rot="R180"/>
 <attribute name="VALUE" x="193.04" y="152.908" size="1.778" layer="96" ratio="12" rot="R180"/>
+<attribute name="DIGIKEY" x="190.5" y="149.86" size="1.778" layer="96" rot="R90" display="off"/>
+<attribute name="MPN" x="190.5" y="149.86" size="1.778" layer="96" rot="R90" display="off"/>
 </instance>
 <instance part="J4" gate="G$1" x="203.2" y="149.86" smashed="yes">
@@
 <attribute name="NAME" x="228.6" y="149.352" size="1.778" layer="95" ratio="12" rot="R180"/>
 <attribute name="VALUE" x="228.6" y="152.908" size="1.778" layer="96" ratio="12" rot="R180"/>
+<attribute name="DIGIKEY" x="226.06" y="149.86" size="1.778" layer="96" rot="R90" display="off"/>
+<attribute name="MPN" x="226.06" y="149.86" size="1.778" layer="96" rot="R90" display="off"/>
 </instance>
 <instance part="L1" gate="G$1" x="215.9" y="137.16" smashed="yes" rot="R180">
 <attribute name="NAME" x="216.408" y="139.7" size="1.778" layer="95" ratio="12" rot="R270"/>
 <attribute name="VALUE" x="212.852" y="139.7" size="1.778" layer="96" ratio="12" rot="R270"/>
+<attribute name="DIGIKEY" x="215.9" y="137.16" size="1.778" layer="96" rot="R180" display="off"/>
+<attribute name="MPN" x="215.9" y="137.16" size="1.778" layer="96" rot="R180" display="off"/>
 </instance>
 <instance part="GND38" gate="1" x="48.26" y="38.1" smashed="yes">

Commit message: mpn and digikey
Parts:
- ANT1: DIGIKEY (none) -> WM15009CT-ND; MPN (none) -> 1462350001
- U13: DIGIKEY (none) -> 296-28299-1-ND; MPN (none) -> TPD3F303DPVR
- U4: DIGIKEY (none) -> BGA725L6E6327FTSA1CT-ND; MANUFACTURER (none) -> Infineon Technologies; MPN (none) -> BGA725L6E6327FTSA1
- U5: DIGIKEY (none) -> 1490-1076-1-ND; MANUFACTURER (none) -> Nordic Semiconductor; MPN (none) -> NRF9160-SICA-R7
Changed lines of the file:
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@@
 <?xml version="1.0" encoding="utf-8"?>
 <!DOCTYPE eagle SYSTEM "eagle.dtd">
-<eagle version="9.5.0">
+<eagle version="9.6.1">
 <drawing>
 <settings>
@@
 <part name="J4" library="connector" deviceset="U.FL-R-SMT" device=""/>
 <part name="GND28" library="supply1" library_urn="urn:adsk.eagle:library:371" deviceset="GND" device=""/>
-<part name="ANT1" library="chips" deviceset="1462350001" device=""/>
+<part name="ANT1" library="chips" deviceset="1462350001" device="">
+<attribute name="DIGIKEY" value="WM15009CT-ND"/>
+<attribute name="MPN" value="1462350001"/>
+</part>
 <part name="BAT1" library="batteries" deviceset="2477THMCOINCELLCLIP" device=""/>
 <part name="GND32" library="supply1" library_urn="urn:adsk.eagle:library:371" deviceset="GND" device=""/>
-<part name="U5" library="chips" deviceset="NRF9160" device=""/>
+<part name="U5" library="chips" deviceset="NRF9160" device="">
+<attribute name="DIGIKEY" value="1490-1076-1-ND"/>
+<attribute name="MANUFACTURER" value="Nordic Semiconductor"/>
+<attribute name="MPN" value="NRF9160-SICA-R7"/>
+</part>
 <part name="C20" library="passives" deviceset="CAPACITOR" device="0402_CAP" value="DNP"/>
 <part name="C21" library="passives" deviceset="CAPACITOR" device="0402_CAP" value="DNP"/>
 <part name="GND33" library="supply1" library_urn="urn:adsk.eagle:library:371" deviceset="GND" device=""/>
-<part name="U4" library="chips" deviceset="BGA725L6" device=""/>
+<part name="U4" library="chips" deviceset="BGA725L6" device="">
+<attribute name="DIGIKEY" value="BGA725L6E6327FTSA1CT-ND"/>
+<attribute name="MANUFACTURER" value=" Infineon Technologies"/>
+<attribute name="MPN" value="BGA725L6E6327FTSA1"/>
+</part>
 <part name="L2" library="passives" deviceset="INDUCTOR" device="0402" value="5.1nH">
 <attribute name="DIGIKEY" value="490-6564-1-ND"/>
@@
 <part name="TP31" library="headers" deviceset="TEST-POINT" device=""/>
 <part name="TP32" library="headers" deviceset="TEST-POINT" device=""/>
-<part name="U13" library="chips" deviceset="TPD3F303DPVR" device=""/>
+<part name="U13" library="chips" deviceset="TPD3F303DPVR" device="">
+<attribute name="DIGIKEY" value="296-28299-1-ND"/>
+<attribute name="MPN" value="TPD3F303DPVR"/>
+</part>
 <part name="GND38" library="supply1" library_urn="urn:adsk.eagle:library:371" deviceset="GND" device=""/>
 <part name="GND39" library="supply1" library_urn="urn:adsk.eagle:library:371" deviceset="GND" device=""/>
@@
 <attribute name="NAME" x="228.86041875" y="165.869590625" size="1.27291875" layer="95"/>
 <attribute name="VALUE" x="228.7332" y="163.83295" size="1.27295" layer="96"/>
+<attribute name="DIGIKEY" x="238.76" y="162.56" size="1.778" layer="96" display="off"/>
+<attribute name="MPN" x="238.76" y="162.56" size="1.778" layer="96" display="off"/>
 </instance>
 <instance part="GND32" gate="1" x="88.9" y="43.18" smashed="yes" rot="R90">
@@
 <attribute name="NAME" x="58.42" y="144.78" size="1.778" layer="95"/>
 <attribute name="VALUE" x="58.42" y="88.9" size="1.778" layer="96"/>
+<attribute name="DIGIKEY" x="96.52" y="121.92" size="1.778" layer="96" display="off"/>
+<attribute name="MANUFACTURER" x="96.52" y="121.92" size="1.778" layer="96" display="off"/>
+<attribute name="MPN" x="96.52" y="121.92" size="1.778" layer="96" display="off"/>
 </instance>
 <instance part="C20" gate="G$1" x="154.94" y="124.46" smashed="yes" rot="R180">
@@
 <attribute name="NAME" x="177.8" y="133.35" size="1.778" layer="95" rot="R180"/>
 <attribute name="VALUE" x="177.8" y="170.18" size="1.778" layer="96" rot="MR0"/>
+<attribute name="DIGIKEY" x="167.64" y="149.86" size="1.778" layer="96" rot="R180" display="off"/>
+<attribute name="MPN" x="167.64" y="149.86" size="1.778" layer="96" rot="R180" display="off"/>
+<attribute name="MANUFACTURER" x="167.64" y="149.86" size="1.778" layer="96" rot="R180" display="off"/>
 </instance>
 <instance part="L2" gate="G$1" x="226.06" y="149.86" smashed="yes" rot="R90">
@@
 <attribute name="NAME" x="58.7756" y="125.9586" size="2.0828" layer="95" ratio="6" rot="SR0"/>
 <attribute name="VALUE" x="58.1406" y="100.5586" size="2.0828" layer="96" ratio="6" rot="SR0"/>
+<attribute name="DIGIKEY" x="50.8" y="119.38" size="1.778" layer="96" display="off"/>
+<attribute name="MPN" x="50.8" y="119.38" size="1.778" layer="96" display="off"/>
 </instance>
 <instance part="P+13" gate="VCC" x="60.96" y="88.9" smashed="yes">

Commit message: renumber
Parts:
- removed TP30: TEST-POINT, headers:TEST-POINT
- added TP24: TEST-POINT, headers:TEST-POINT
- C16: DESCRIPTION CAP CER 4.7UF 10V X5R 0402 -> (none); DIGIKEY 1276-1480-1-ND -> 445-5947-1-ND; MANUFACTURER Samsung Electro-Mechanics -> (none); MPN CL05A475KP5NRNC -> C1005X5R0J475K050BC
- J1: value TC2030-JLINK-NL -> DM3AT-SF-PEJM5; device connector:TC2030-JLINK-NL -> connector:DM3AT-SF-PEJM5
- J2: value U.FL-R-SMT -> NANO_SIM; device connector:U.FL-R-SMT -> signpost:NANO_SIM
- J3: value NANO_SIM -> TC2030-JLINK-NL; device signpost:NANO_SIM -> connector:TC2030-JLINK-NL
- J5: value DM3AT-SF-PEJM5 -> U.FL-R-SMT; device connector:DM3AT-SF-PEJM5 -> connector:U.FL-R-SMT
- R11, R12, R13: DESCRIPTION RES SMD 10K OHM 1% 1/16W 0402 -> (none); DIGIKEY 1276-3431-1-ND -> 311-10KJRCT-ND; MANUFACTURER Samsung Electro-Mechanics -> (none); MPN RC1005F103CS -> RC0402JR-0710KL
- U10: value SIP32510 -> SI7021-A20-GM1; device chips:SIP32510 -> chips:SI7021-A20-GM1; DESCRIPTION IC LOAD SWITCH SOT23-6 -> (none); MPN (none) -> SI7021-A20-GM1
- U11: value SI7021-A20-GM1 -> SIP32510; device chips:SI7021-A20-GM1 -> chips:SIP32510; DESCRIPTION (none) -> IC LOAD SWITCH SOT23-6; MPN SI7021-A20-GM1 -> (none)
- U2: value BQ25505 -> BGA725L6; device chips:BQ25505 -> chips:BGA725L6; DIGIKEY (none) -> BGA725L6E6327FTSA1CT-ND; MANUFACTURER (none) -> Infineon Technologies; MPN (none) -> BGA725L6E6327FTSA1
- U3: value EKMB1101111 -> BQ25505; device chips:EKMB1101111 -> chips:BQ25505
- U4: value BGA725L6 -> EKMB1101111; device chips:BGA725L6 -> chips:EKMB1101111; DIGIKEY BGA725L6E6327FTSA1CT-ND -> (none); MANUFACTURER Infineon Technologies -> (none); MPN BGA725L6E6327FTSA1 -> (none)
- U5: value NRF9160 -> LIS2DW12; device chips:NRF9160 -> chips:LIS2DW12; DIGIKEY 1490-1076-1-ND -> (none); MANUFACTURER Nordic Semiconductor -> (none); MPN NRF9160-SICA-R7 -> (none)
- U6: value LIS2DW12 -> MAX17222; device chips:LIS2DW12 -> chips:MAX17222
- U7: value MAX17222 -> MAX44009; device chips:MAX17222 -> chips:MAX44009
- U8: value MAX44009 -> MS5637-02BA03; device chips:MAX44009 -> chips:MS5637-02BA03
- U9: value MS5637-02BA03 -> NRF9160; device chips:MS5637-02BA03 -> chips:NRF9160; DIGIKEY (none) -> 1490-1076-1-ND; MANUFACTURER (none) -> Nordic Semiconductor; MPN (none) -> NRF9160-SICA-R7
- renumbered BAT1 to BT2, Q10 to Q9, TP31 to TP28, TP32 to TP29, X4 to X1
Connections:
- net !CLR_EN: now also U9.P0.08; no longer U5.P0.08
- net !CLR_INT: now also U9.P0.29; no longer U5.P0.29
- net !HUM_EN: now also U9.P0.04; no longer U5.P0.04
- net !LT_EN: now also U9.P0.30; no longer U5.P0.30
- net !LT_INT: now also U7.!INT, U9.P0.02; no longer U5.P0.02, U8.!INT
- net !PIR_EN: now also U9.P0.24; no longer U5.P0.24
- net !PR_EN: now also U9.P0.23; no longer U5.P0.23
- net !RST: now also J3.!RESET, U9.NRESSET; no longer J1.!RESET, U5.NRESSET
- net !RTC_IRQ1: now also U9.P0.11; no longer U5.P0.11
- net !RTC_IRQ2: now also U9.P0.10; no longer U5.P0.10
- net !RTC_IRQ3: now also U9.P0.09; no longer U5.P0.09
- net !SD_CS: now also J1.DATA3-CD/CS_N, U9.P0.26; no longer J5.DATA3-CD/CS_N, U5.P0.26
- net !SD_DETECT: now also J1.A, U9.P0.27; no longer J5.A, U5.P0.27
- net !VBAT_PRI_ON: now also U3.!VBAT_PRI_ON; no longer U2.!VBAT_PRI_ON
- net !VBAT_SEC_ON: now also U3.!VBAT_SEC_ON; no longer U2.!VBAT_SEC_ON
- net ACC_CS: now also U5.CS, U9.P0.06; no longer U5.P0.06, U6.CS
- net ACC_INT1: now also U5.INT1, U9.P0.05; no longer U5.P0.05, U6.INT1
- net ACC_INT2: now also U5.INT2, U9.P0.07; no longer U5.P0.07, U6.INT2
- net GND: now also J1.B, J2.C5(GND), J3.GND, J5.P$2, TP26.TESTPOINT, U2.GND@1, U2.GND@4, U3.!EN, U4.GND, U7.A0; no longer J2.P$2, J3.C5(GND), J5.B, J5.GND, TP27.TESTPOINT, U2.!EN, U2.GND, U4.GND@1, U4.GND@4, U8.A0
- net GPS_EN: now also U2.PON, U9.MAGPIO0; no longer U4.PON, U5.MAGPIO0
- net LBST: now also U3.LBST; no longer U2.LBST
- net LED_BLUE: now also U9.P0.17; no longer U5.P0.17
- net LED_GREEN: now also U9.P0.19; no longer U5.P0.19
- net LED_RED: now also U9.P0.18; no longer U5.P0.18
- net MISO: now also J1.DATA0/MISO, U5.MISO/SA0, U9.P0.22; no longer J5.DATA0/MISO, U5.P0.22, U6.MISO/SA0
- net MOSI: now also J1.CMD/MOSI, U5.MOSI/SDA, U9.P0.21; no longer J5.CMD/MOSI, U5.P0.21, U6.MOSI/SDA
- net N$1: now also U2.AO, U9.GPS; no longer U4.AO, U5.GPS
- net N$12: now also U6.SEL; no longer U7.SEL
- net N$13: now also J1.VCC, U11.VLOAD; no longer J5.VCC, U10.VLOAD
- net N$14: now also U6.EN; no longer U7.EN
- net N$18: now also U3.VBAT_OV; no longer U2.VBAT_OV
- net N$2: now also U2.AI; no longer U4.AI
- net N$20: now also U7.VCC; no longer U8.VCC
- net N$21: now also U8.VDD; no longer U9.VDD
- net N$22: now also U10.VCC; no longer U11.VCC
- net N$23: now also U4.VCC; no longer U3.VCC
- net N$28: now also U9.ENABLE; no longer U5.ENABLE
- net N$29: now also U9.IO_SUPPLY; no longer U5.IO_SUPPLY
- net N$32: now also U3.VRDIV; no longer U2.VRDIV
- net N$34: now also U8.SCL; no longer U9.SCL
- net N$4: now also J5.ANT; no longer J4.ANT
- net N$41: now also U8.SDA; no longer U9.SDA
- net N$48: now also U10.SDA; no longer U11.SDA
- net N$50: now also U10.SCL; no longer U11.SCL
- net N$51: now also U7.SDA; no longer U8.SDA
- net N$52: now also U7.SCL; no longer U8.SCL
- net N$57: now also U3.OK_PROG; no longer U2.OK_PROG
- net N$58: now also U3.OK_HYST; no longer U2.OK_HYST
- net N$8: now also J4.ANT, U9.ANT; no longer J2.ANT, U5.ANT
- net PIR_OUT: now also U4.OUT, U9.P0.25; no longer U3.OUT, U5.P0.25
- net RTC_CS: now also U9.P0.12; no longer U5.P0.12
- net SCK: now also J1.CLK, U5.SCL/SPC, U9.P0.03; no longer J5.CLK, U5.P0.03, U6.SCL/SPC
- net SCL: now also U9.P0.01; no longer U5.P0.01
- net SDA: now also U9.P0.00; no longer U5.P0.00
- net SD_ENABLE: now also U11.EN, U9.P0.28; no longer U10.EN, U5.P0.28
- net SIM_1V8: now also J2.C1(VCC), U9.SIM_1V8; no longer J3.C1(VCC), U5.SIM_1V8
- net SIM_CLK: now also U9.SIM_CLK; no longer U5.SIM_CLK
- net SIM_CLK2: now also J2.C3(CLK); no longer J3.C3(CLK)
- net SIM_IO: now also U9.SIM_IO; no longer U5.SIM_IO
- net SIM_IO2: now also J2.C7(IO); no longer J3.C7(IO)
- net SIM_RST: now also U9.SIM_RST; no longer U5.SIM_RST
- net SIM_RST2: now also J2.C2(RST), TP27.TESTPOINT; no longer J3.C2(RST), TP30.TESTPOINT
- net SW: now also TP24.TESTPOINT, U6.LX; no longer TP25.TESTPOINT, U7.LX
- net SWDCLK: now also J3.SWDCLK, U9.SWD_CLK; no longer J1.SWDCLK, U5.SWD_CLK
- net SWDIO: now also J3.SWDIO, U9.SWD_IO; no longer J1.SWDIO, U5.SWD_IO
- net VBAT: now also U3.VBAT_PRI, U9.P0.15; no longer U2.VBAT_PRI, U5.P0.15
- net VBAT_OK: now also U3.VBAT_OK, U9.P0.20; no longer U2.VBAT_OK, U5.P0.20
- net VCC: now also J3.VCC, TP25.TESTPOINT, U11.VSUPP, U2.VCC, U5.VCC, U5.VDD_IO, U6.OUT, U9.VDD, U9.VDD_GPIO; no longer J1.VCC, TP26.TESTPOINT, U10.VSUPP, U4.VCC, U5.VDD, U5.VDD_GPIO, U6.VCC, U6.VDD_IO, U7.OUT
- net VOC_SAMP_VSTOR: now also U3.VOC_SAMP, U3.VSTOR; no longer U2.VOC_SAMP, U2.VSTOR
- net VREF_SAMP: now also U3.VREF_SAMP; no longer U2.VREF_SAMP
- net VSEC: now also U3.VBAT_SEC, U9.P0.13; no longer U2.VBAT_SEC, U5.P0.13
- net VSOL: now also U3.VIN_DC, U9.P0.14; no longer U2.VIN_DC, U5.P0.14
- net VSW: now also U6.IN; no longer U7.IN
- net WDI: now also U9.P0.16; no longer U5.P0.16
Other:
- moved on the sheet: J4, TP25, TP26

Commit message: remove tp and jlink from bom
Parts:
- C16: MPN C1005X5R0J475K050BC -> C1005X5R0J475K050BC
- R11, R12, R13: DIGIKEY 311-10KJRCT-ND -> 311-10KJRCT-ND
Changed lines of the file:
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@@
 <part name="C16" library="passives" deviceset="CAPACITOR" device="0402_CAP" value="4.7uF">
 <attribute name="DIGIKEY" value="445-5947-1-ND"/>
-<attribute name="MPN" value="C1005X5R0J475K050BC"/>
+<attribute name="MPN" value="C1005X5R0J475K050BC "/>
 </part>
 <part name="GND37" library="umich" deviceset="GND" device=""/>
 <part name="J1" library="connector" deviceset="DM3AT-SF-PEJM5" device=""/>
 <part name="R11" library="passives" deviceset="RESISTOR" device="0402_RES" value="10k">
-<attribute name="DIGIKEY" value="311-10KJRCT-ND"/>
+<attribute name="DIGIKEY" value="311-10KJRCT-ND "/>
 <attribute name="MPN" value="RC0402JR-0710KL"/>
 </part>
 <part name="R12" library="passives" deviceset="RESISTOR" device="0402_RES" value="10k">
-<attribute name="DIGIKEY" value="311-10KJRCT-ND"/>
+<attribute name="DIGIKEY" value="311-10KJRCT-ND "/>
 <attribute name="MPN" value="RC0402JR-0710KL"/>
 </part>
 <part name="R13" library="passives" deviceset="RESISTOR" device="0402_RES" value="10k">
-<attribute name="DIGIKEY" value="311-10KJRCT-ND"/>
+<attribute name="DIGIKEY" value="311-10KJRCT-ND "/>
 <attribute name="MPN" value="RC0402JR-0710KL"/>
 </part>
